Commit message: Add pickup truck urdf.

File: smarts/assets/vehicles/dynamics_model/generic_pickup_truck.urdf (robot description, URDF)
Before this commit: robot vehicle, 10 links, 9 joints
Links:
- removed link box
- removed link cab
- link chassis: geometry collision box size=1.91 5.0 1.89; visual box size=1.91 5.0 1.89
- link front_left_wheel: geometry collision cylinder length=0.35 radius=0.47; visual cylinder length=0.35 radius=0.47
- link front_right_wheel: geometry collision cylinder length=0.35 radius=0.47; visual cylinder length=0.35 radius=0.47
- link rear_left_wheel: geometry collision cylinder length=0.35 radius=0.47; visual cylinder length=0.35 radius=0.47
- link rear_right_wheel: geometry collision cylinder length=0.35 radius=0.47; visual cylinder length=0.35 radius=0.47
Joints:
- removed joint box_link_connection
- removed joint cab_link_connection
- joint front_left_steer_joint: origin xyz=1.0 -2.5 0.5 rpy=0 0 0 -> xyz=0.5 -1.88 0.5 rpy=0 0 0
- joint front_right_steer_joint: origin xyz=-1.0 -2.5 0.5 rpy=0 0 0 -> xyz=-0.5 -1.88 0.5 rpy=0 0 0
- joint rear_left_wheel_joint: origin xyz=0.845 2.5 0.5 rpy=0 0 0 -> xyz=0.7 1.35 0.5 rpy=0 0 0
- joint rear_right_wheel_joint: origin xyz=-0.845 2.5 0.5 rpy=0 0 0 -> xyz=-0.7 1.35 0.5 rpy=0 0 0
