Commit message: Update to final vehicle set.

File: smarts/assets/vehicles/dynamics_model/generic_class_2a_truck.urdf (robot description, URDF)
Before this commit: robot vehicle, 10 links, 9 joints
Links:
- removed link box
- removed link cab
- link chassis: mass 2000.0 -> 3000.0; geometry collision box size=1.91 5.0 1.89; visual box size=1.91 5.0 1.89
- link front_left_wheel: geometry collision cylinder length=0.35 radius=0.47; visual cylinder length=0.35 radius=0.47
- link front_right_wheel: geometry collision cylinder length=0.35 radius=0.47; visual cylinder length=0.35 radius=0.47
- link rear_left_wheel: geometry collision cylinder length=0.35 radius=0.47; visual cylinder length=0.35 radius=0.47
- link rear_right_wheel: geometry collision cylinder length=0.35 radius=0.47; visual cylinder length=0.35 radius=0.47
Joints:
- removed joint box_link_connection
- removed joint cab_link_connection
- joint front_left_steer_joint: origin xyz=0.95 -2.5 0.5 rpy=0 0 0 -> xyz=0.5 -1.88 0.5 rpy=0 0 0
- joint front_right_steer_joint: origin xyz=-0.95 -2.5 0.5 rpy=0 0 0 -> xyz=-0.5 -1.88 0.5 rpy=0 0 0
- joint rear_left_wheel_joint: origin xyz=0.84 2.5 0.5 rpy=0 0 0 -> xyz=0.7 1.35 0.5 rpy=0 0 0
- joint rear_right_wheel_joint: origin xyz=-0.84 2.5 0.5 rpy=0 0 0 -> xyz=-0.7 1.35 0.5 rpy=0 0 0

File: smarts/assets/vehicles/dynamics_model/generic_class_5_truck_empty.urdf (robot description, URDF)
Before this commit: robot vehicle, 8 links, 7 joints
Links:
- added link box, mass 500.0; visual box size=2.3 5.05 2.05
- added link cab, mass 2500.0; visual box size=2.0 1.8 2.0
- link chassis: mass 2000.0 -> 3500.0; geometry collision box size=2.4 7.1 2.4; visual box size=2.4 7.1 2.4
- link front_left_wheel: geometry collision cylinder length=0.35 radius=0.52; visual cylinder length=0.35 radius=0.52
- link front_right_wheel: geometry collision cylinder length=0.35 radius=0.52; visual cylinder length=0.35 radius=0.52
- link rear_left_wheel: geometry collision cylinder length=0.7 radius=0.52; visual cylinder length=0.7 radius=0.52
- link rear_right_wheel: geometry collision cylinder length=0.7 radius=0.52; visual cylinder length=0.7 radius=0.52
Joints:
- added joint box_link_connection: type fixed, parent chassis, child box, origin xyz=0 0.9 0.15 rpy=0 0 3.141592653589793
- added joint cab_link_connection: type fixed, parent chassis, child cab, origin xyz=0 -2.60 0 rpy=0 0 3.141592653589793
- joint front_left_steer_joint: origin xyz=0.5 -1.88 0.5 rpy=0 0 0 -> xyz=0.95 -2.5 0.5 rpy=0 0 0
- joint front_right_steer_joint: origin xyz=-0.5 -1.88 0.5 rpy=0 0 0 -> xyz=-0.95 -2.5 0.5 rpy=0 0 0
- joint rear_left_wheel_joint: origin xyz=0.7 1.35 0.5 rpy=0 0 0 -> xyz=0.84 2.5 0.5 rpy=0 0 0
- joint rear_right_wheel_joint: origin xyz=-0.7 1.35 0.5 rpy=0 0 0 -> xyz=-0.84 2.5 0.5 rpy=0 0 0

File: smarts/assets/vehicles/dynamics_model/generic_class_5_truck_loaded.urdf (robot description, URDF)
Before this commit: robot vehicle, 10 links, 9 joints
Links:
- link box: mass 1500.0 -> 2700.0
- link cab: mass 3000.0 -> 2500.0
- link chassis: mass 2000.0 -> 3500.0
